File: proyectosKicad/calidadAire/calidadAire.kicad_pcb (KiCad board)
At the start: 2 copper layers, 15 parts, among them J1 test_ADC, J2 DHT11, J3 GND, J4 5V, P1 POLVO, P2 ADC, P3 GAS, P4 GPS, Q1 PN2222A, U1 UnloquerMCU_ver01

Commit message: ruteada tarjeta calidad aire, revisar footprint capacitor, muy pequeno
Parts:
- added C1: CP, Capacitors_ThroughHole:CP_Axial_L10.0mm_D4.5mm_P15.00mm_Horizontal, F.Cu at (241.3, 73.6)
- added C1: CP, Capacitors_ThroughHole:CP_Axial_L10.0mm_D4.5mm_P15.00mm_Horizontal, F.Cu at (101.6, 153.9)
- added J1: test_ADC, Pin_Headers:Pin_Header_Straight_1x10_Pitch2.54mm, F.Cu at (193.3, 85.3)
- added J1: test_ADC, Pin_Headers:Pin_Header_Straight_1x10_Pitch2.54mm, F.Cu at (53.6, 165.6)
- added J2: DHT11, Pin_Headers:Pin_Header_Straight_1x04_Pitch2.54mm, F.Cu at (223.4, 86.5)
- added J2: DHT11, Pin_Headers:Pin_Header_Straight_1x04_Pitch2.54mm, F.Cu at (83.7, 166.8)
- added J3: GND, Pin_Headers:Pin_Header_Straight_1x03_Pitch2.54mm, F.Cu at (207.8, 40.4)
- added J3: GND, Pin_Headers:Pin_Header_Straight_1x03_Pitch2.54mm, F.Cu at (68.1, 120.7)
- added J4: 5V, Pin_Headers:Pin_Header_Straight_1x03_Pitch2.54mm, F.Cu at (207.7, 45.9)
- added J4: 5V, Pin_Headers:Pin_Header_Straight_1x03_Pitch2.54mm, F.Cu at (68.0, 126.2)
- added P1: POLVO, footprints_unloquer:sensor_polvo, F.Cu at (249.2, 45.3)
- added P1: POLVO, footprints_unloquer:sensor_polvo, F.Cu at (109.5, 125.6)
- added P2: ADC, footprints_unloquer:ads1115, F.Cu at (205.7, 100.6)
- added P2: ADC, footprints_unloquer:ads1115, F.Cu at (66.0, 180.8)
- added P3: GAS, Pin_Headers:Pin_Header_Straight_1x03_Pitch2.54mm, F.Cu at (179.3, 91.8)
- added P3: GAS, Pin_Headers:Pin_Header_Straight_1x03_Pitch2.54mm, F.Cu at (39.6, 172.1)
- added P4: GPS, footprints_unloquer:gps, F.Cu at (178.3, 64.8)
- added P4: GPS, footprints_unloquer:gps, F.Cu at (38.6, 145.0)
- added Q1: PN2222A, TO_SOT_Packages_THT:TO-92_Molded_Narrow, F.Cu at (232.9, 56.1)
- added Q1: PN2222A, TO_SOT_Packages_THT:TO-92_Molded_Narrow, F.Cu at (93.2, 136.3)
- added R1: R, Resistors_ThroughHole:R_Axial_DIN0204_L3.6mm_D1.6mm_P2.54mm_Vertical, F.Cu at (226.4, 54.5)
- added R1: R, Resistors_ThroughHole:R_Axial_DIN0204_L3.6mm_D1.6mm_P2.54mm_Vertical, F.Cu at (86.7, 134.7)
- added R2: R, Resistors_ThroughHole:R_Axial_DIN0204_L3.6mm_D1.6mm_P2.54mm_Vertical, F.Cu at (233.2, 50.5)
- added R2: R, Resistors_ThroughHole:R_Axial_DIN0204_L3.6mm_D1.6mm_P2.54mm_Vertical, F.Cu at (93.5, 130.8)
- added R3: R, Resistors_ThroughHole:R_Axial_DIN0204_L3.6mm_D1.6mm_P2.54mm_Vertical, F.Cu at (236.2, 68.9)
- added R3: R, Resistors_ThroughHole:R_Axial_DIN0204_L3.6mm_D1.6mm_P2.54mm_Vertical, F.Cu at (96.5, 149.1)
- added R4: R, Resistors_ThroughHole:R_Axial_DIN0204_L3.6mm_D1.6mm_P2.54mm_Vertical, F.Cu at (228.4, 80.6)
- added R4: R, Resistors_ThroughHole:R_Axial_DIN0204_L3.6mm_D1.6mm_P2.54mm_Vertical, F.Cu at (88.7, 160.9)
- added U1: UnloquerMCU_ver01, unloqueMCU_ver01_footprint:UnloquerMCU_ver01_footprint, F.Cu at (204.0, 62.4)
- added U1: UnloquerMCU_ver01, unloqueMCU_ver01_footprint:UnloquerMCU_ver01_footprint, F.Cu at (64.3, 142.6)
- moved R2 100.9 mm to (93.0, 38.8)
- moved J2 98.3 mm to (83.2, 74.8)
- moved J1 98.3 mm to (53.1, 73.7)
- moved P2 98.3 mm to (65.5, 88.9)
- moved P4 98.3 mm to (38.1, 53.1)
- moved Q1 98.3 mm to (92.7, 44.4)
- moved R1 98.3 mm to (86.2, 42.8)
- moved U1 98.3 mm to (63.8, 50.7)
- moved P1 98.3 mm to (109.0, 33.6)
- moved P3 98.3 mm to (39.1, 80.2)
- moved R3 98.3 mm to (96.0, 57.2)
- moved R4 98.3 mm to (88.2, 68.9)
- moved J3 95.0 mm to (67.6, 28.7)
- moved C1 93.4 mm to (101.1, 62.0), turned to 180 degrees
- moved J4 86.9 mm to (67.5, 34.3)
Routing:
- net /GND: track 99.2 -> 740.0 mm
- net /5V: track 71.9 -> 586.7 mm
- net /A1: track 68.4 -> 205.2 mm
- net /gpio5: track 35.6 -> 130.1 mm
- net /GPIO0: track 30.7 -> 114.3 mm
- net /gpio4: track 41.2 -> 123.6 mm
- net /polvo_1: track 31.5 -> 106.5 mm
- net /A0: track 35.6 -> 106.8 mm
- net /GPIO16: track 28.5 -> 85.5 mm
- net /gpio15: track 24.5 -> 73.4 mm
- net /P3: track 19.6 -> 47.5 mm
- net /gpio2: track 12.4 -> 37.1 mm
- net Net-(J1-Pad1): track 7.73 -> 23.2 mm
- net Net-(J1-Pad2): track 7.73 -> 23.2 mm
- net Net-(Q1-Pad2): track 5.61 -> 16.8 mm
- added copper zone on F.Cu, net /GND
Other:
- board outline added: 258.5 x 173.4 mm
