File: proyectosKicad/calidadAire/calidadAire.kicad_pcb (KiCad board)
At the start: 2 copper layers, 258.5 x 173.4 mm, 45 parts, among them J1 test_ADC, J2 DHT11, J3 GND, J4 5V, P1 POLVO, P2 ADC, P3 GAS, P4 GPS, Q1 PN2222A, U1 UnloquerMCU_ver01

Commit message: footprint de transistor mas grande
Parts:
- removed the C1 at (241.3, 73.6)
- removed the C1 at (101.6, 153.9)
- removed the J1 at (193.3, 85.3)
- removed the J1 at (53.6, 165.6)
- removed the J2 at (223.4, 86.5)
- removed the J2 at (83.7, 166.8)
- removed the J3 at (207.8, 40.4)
- removed the J3 at (68.1, 120.7)
- removed the J4 at (207.7, 45.9)
- removed the J4 at (68.0, 126.2)
- removed the P1 at (249.2, 45.3)
- removed the P1 at (109.5, 125.6)
- removed the P2 at (205.7, 100.6)
- removed the P2 at (66.0, 180.8)
- removed the P3 at (179.3, 91.8)
- removed the P3 at (39.6, 172.1)
- removed the P4 at (178.3, 64.8)
- removed the P4 at (38.6, 145.0)
- removed the Q1 at (232.9, 56.1)
- removed the Q1 at (93.2, 136.3)
- removed the Q1 at (92.7, 44.4)
- removed the R1 at (226.4, 54.5)
- removed the R1 at (86.7, 134.7)
- removed the R2 at (233.2, 50.5)
- removed the R2 at (93.5, 130.8)
- removed the R3 at (236.2, 68.9)
- removed the R3 at (96.5, 149.1)
- removed the R4 at (228.4, 80.6)
- removed the R4 at (88.7, 160.9)
- removed the U1 at (204.0, 62.4)
- removed the U1 at (64.3, 142.6)
- added C1: CP, Capacitors_ThroughHole:CP_Axial_L10.0mm_D4.5mm_P15.00mm_Horizontal, F.Cu at (234.2, 67.0)
- added C1: CP, Capacitors_ThroughHole:CP_Axial_L10.0mm_D4.5mm_P15.00mm_Horizontal, F.Cu at (105.1, 156.2)
- added J1: test_ADC, Pin_Headers:Pin_Header_Straight_1x10_Pitch2.54mm, F.Cu at (186.2, 78.7)
- added J1: test_ADC, Pin_Headers:Pin_Header_Straight_1x10_Pitch2.54mm, F.Cu at (57.1, 167.9)
- added J2: DHT11, Pin_Headers:Pin_Header_Straight_1x04_Pitch2.54mm, F.Cu at (216.3, 79.9)
- added J2: DHT11, Pin_Headers:Pin_Header_Straight_1x04_Pitch2.54mm, F.Cu at (87.2, 169.1)
- added J3: GND, Pin_Headers:Pin_Header_Straight_1x03_Pitch2.54mm, F.Cu at (200.6, 33.8)
- added J3: GND, Pin_Headers:Pin_Header_Straight_1x03_Pitch2.54mm, F.Cu at (71.6, 123.0)
- added J4: 5V, Pin_Headers:Pin_Header_Straight_1x03_Pitch2.54mm, F.Cu at (200.6, 39.3)
- added J4: 5V, Pin_Headers:Pin_Header_Straight_1x03_Pitch2.54mm, F.Cu at (71.5, 128.5)
- added P1: POLVO, footprints_unloquer:sensor_polvo, F.Cu at (242.1, 38.7)
- added P1: POLVO, footprints_unloquer:sensor_polvo, F.Cu at (113.0, 127.9)
- added P2: ADC, footprints_unloquer:ads1115, F.Cu at (198.6, 94.0)
- added P2: ADC, footprints_unloquer:ads1115, F.Cu at (69.5, 183.1)
- added P3: GAS, Pin_Headers:Pin_Header_Straight_1x03_Pitch2.54mm, F.Cu at (172.2, 85.2)
- added P3: GAS, Pin_Headers:Pin_Header_Straight_1x03_Pitch2.54mm, F.Cu at (43.1, 174.4)
- added P4: GPS, footprints_unloquer:gps, F.Cu at (171.2, 58.2)
- added P4: GPS, footprints_unloquer:gps, F.Cu at (42.1, 147.3)
- added Q1: PN2222A, TO_SOT_Packages_THT:TO-92_Molded_Wide, F.Cu at (225.8, 49.5)
- added Q1: PN2222A, TO_SOT_Packages_THT:TO-92_Molded_Wide, F.Cu at (96.7, 138.6)
- added Q1: PN2222A, TO_SOT_Packages_THT:TO-92_Molded_Wide, F.Cu at (92.7, 44.4)
- added R1: R, Resistors_ThroughHole:R_Axial_DIN0204_L3.6mm_D1.6mm_P2.54mm_Vertical, F.Cu at (219.3, 47.9)
- added R1: R, Resistors_ThroughHole:R_Axial_DIN0204_L3.6mm_D1.6mm_P2.54mm_Vertical, F.Cu at (90.2, 137.0)
- added R2: R, Resistors_ThroughHole:R_Axial_DIN0204_L3.6mm_D1.6mm_P2.54mm_Vertical, F.Cu at (226.1, 43.9)
- added R2: R, Resistors_ThroughHole:R_Axial_DIN0204_L3.6mm_D1.6mm_P2.54mm_Vertical, F.Cu at (97.0, 133.1)
- added R3: R, Resistors_ThroughHole:R_Axial_DIN0204_L3.6mm_D1.6mm_P2.54mm_Vertical, F.Cu at (229.1, 62.3)
- added R3: R, Resistors_ThroughHole:R_Axial_DIN0204_L3.6mm_D1.6mm_P2.54mm_Vertical, F.Cu at (100.0, 151.4)
- added R4: R, Resistors_ThroughHole:R_Axial_DIN0204_L3.6mm_D1.6mm_P2.54mm_Vertical, F.Cu at (221.3, 74.0)
- added R4: R, Resistors_ThroughHole:R_Axial_DIN0204_L3.6mm_D1.6mm_P2.54mm_Vertical, F.Cu at (92.2, 163.1)
- added U1: UnloquerMCU_ver01, unloqueMCU_ver01_footprint:UnloquerMCU_ver01_footprint, F.Cu at (196.8, 55.8)
- added U1: UnloquerMCU_ver01, unloqueMCU_ver01_footprint:UnloquerMCU_ver01_footprint, F.Cu at (67.8, 144.9)
Routing:
- net Net-(Q1-Pad2): track 16.8 -> 20.6 mm
- net /P3: track 47.5 -> 50.2 mm
Other:
- board size 258.5 x 173.4 mm -> 251.4 x 175.7 mm
