File: proyectosKicad/calidadAire/calidadAire.sch (KiCad schematic (older format))
At the start: 15 parts, among them J1 test_ADC, J2 DHT11, J3 GND, J4 5V, P1 POLVO, P2 ADC, P3 GAS, P4 GPS, Q1 PN2222A, U1 UnloquerMCU_ver01

Commit message: footprint de transistor mas grande
Parts:
- Q1: footprint TO_SOT_Packages_THT:TO-92_Molded_Narrow -> TO_SOT_Packages_THT:TO-92_Molded_Wide
Changed lines of the file:
@@
 F 0 "Q1" H 2650 3575 50  0000 L CNN
 F 1 "PN2222A" H 2650 3500 50  0000 L CNN
-F 2 "TO_SOT_Packages_THT:TO-92_Molded_Narrow" H 2650 3425 50  0001 L CIN
+F 2 "TO_SOT_Packages_THT:TO-92_Molded_Wide" H 2650 3425 50  0001 L CIN
 F 3 "" H 2450 3500 50  0001 L CNN
 	1    2450 3500
