File: proyectosKicad/calidadAirePlantTower/polvo_sensor_plant_tower.kicad_pcb (KiCad board)
At the start: 2 copper layers, 227.3 x 150.5 mm, 65 parts, among them J1 PLANTTOWER, J2 GPS, J3 DHT, U1 UnloquerMCU_ver01

Commit message: alimentacion y pines ok
Parts:
- removed the J1 at (41.9, 142.9)
- removed the J1 at (91.4, 31.8)
- removed the J1 at (92.1, 87.6)
- removed the J1 at (41.3, 87.0)
- removed the J1 at (92.7, 143.5)
- removed the J1 at (142.9, 144.8)
- removed the J1 at (187.3, 91.4)
- removed the J1 at (186.7, 35.6)
- removed the J1 at (236.9, 36.8)
- removed the J1 at (237.5, 92.7)
- removed the J1 at (142.2, 88.9)
- removed the J1 at (141.6, 33.0)
- removed the J2 at (34.3, 151.1)
- removed the J2 at (83.8, 40.0)
- removed the J2 at (84.5, 95.9)
- removed the J2 at (33.7, 95.2)
- removed the J2 at (85.1, 151.8)
- removed the J2 at (135.3, 153.0)
- removed the J2 at (179.7, 99.7)
- removed the J2 at (179.1, 43.8)
- removed the J2 at (229.2, 45.1)
- removed the J2 at (229.9, 101.0)
- removed the J2 at (134.6, 97.2)
- removed the J2 at (134.0, 41.3)
- removed the J3 at (34.9, 145.4)
- removed the J3 at (84.5, 34.3)
- removed the J3 at (85.1, 90.2)
- removed the J3 at (34.3, 89.5)
- removed the J3 at (85.7, 146.1)
- removed the J3 at (135.9, 147.3)
- removed the J3 at (180.3, 94.0)
- removed the J3 at (179.7, 38.1)
- removed the J3 at (229.9, 39.4)
- removed the J3 at (230.5, 95.2)
- removed the J3 at (135.3, 91.4)
- removed the J3 at (134.6, 35.6)
- removed the R1 at (31.1, 140.3)
- removed the R1 at (80.6, 29.2)
- removed the R1 at (81.3, 85.1)
- removed the R1 at (30.5, 84.5)
- removed the R1 at (81.9, 141.0)
- removed the R1 at (132.1, 142.2)
- removed the R1 at (176.5, 88.9)
- removed the R1 at (175.9, 33.0)
- removed the R1 at (226.1, 34.3)
- removed the R1 at (226.7, 90.2)
- removed the R1 at (131.4, 86.4)
- removed the R1 at (130.8, 30.5)
- removed the U1 at (35.7, 150.8)
- removed the U1 at (85.2, 39.6)
- removed the U1 at (85.8, 95.5)
- removed the U1 at (35.0, 94.9)
- removed the U1 at (86.5, 151.4)
- removed the U1 at (136.6, 152.7)
- removed the U1 at (181.1, 99.3)
- removed the U1 at (180.5, 43.5)
- removed the U1 at (230.6, 44.7)
- removed the U1 at (231.3, 100.6)
- removed the U1 at (136.0, 96.8)
- removed the U1 at (135.4, 40.9)
- added J1: PLANTTOWER, Pin_Headers:Pin_Header_Straight_1x03_Pitch2.54mm, F.Cu at (193.5, 32.6)
- added J1: PLANTTOWER, Pin_Headers:Pin_Header_Straight_1x03_Pitch2.54mm, F.Cu at (148.3, 33.0)
- added J1: PLANTTOWER, Pin_Headers:Pin_Header_Straight_1x03_Pitch2.54mm, F.Cu at (74.4, 31.5)
- added J1: PLANTTOWER, Pin_Headers:Pin_Header_Straight_1x03_Pitch2.54mm, F.Cu at (227.3, 33.0)
- added J1: PLANTTOWER, Pin_Headers:Pin_Header_Straight_1x03_Pitch2.54mm, F.Cu at (227.3, 128.5)
- added J1: PLANTTOWER, Pin_Headers:Pin_Header_Straight_1x03_Pitch2.54mm, F.Cu at (193.5, 128.1)
- added J1: PLANTTOWER, Pin_Headers:Pin_Header_Straight_1x03_Pitch2.54mm, F.Cu at (40.6, 126.6)
- added J1: PLANTTOWER, Pin_Headers:Pin_Header_Straight_1x03_Pitch2.54mm, F.Cu at (74.4, 127.0)
- added J1: PLANTTOWER, Pin_Headers:Pin_Header_Straight_1x03_Pitch2.54mm, F.Cu at (148.3, 128.5)
- added J1: PLANTTOWER, Pin_Headers:Pin_Header_Straight_1x03_Pitch2.54mm, F.Cu at (114.6, 128.1)
- added J1: PLANTTOWER, Pin_Headers:Pin_Header_Straight_1x03_Pitch2.54mm, F.Cu at (114.6, 32.6)
- added J2: GPS, Pin_Headers:Pin_Header_Straight_1x03_Pitch2.54mm, F.Cu at (185.9, 40.9)
- added J2: GPS, Pin_Headers:Pin_Header_Straight_1x03_Pitch2.54mm, F.Cu at (140.7, 41.2)
- added J2: GPS, Pin_Headers:Pin_Header_Straight_1x03_Pitch2.54mm, F.Cu at (66.8, 39.7)
- added J2: GPS, Pin_Headers:Pin_Header_Straight_1x03_Pitch2.54mm, F.Cu at (219.7, 41.2)
- added J2: GPS, Pin_Headers:Pin_Header_Straight_1x03_Pitch2.54mm, F.Cu at (219.7, 136.8)
- added J2: GPS, Pin_Headers:Pin_Header_Straight_1x03_Pitch2.54mm, F.Cu at (185.9, 136.4)
- added J2: GPS, Pin_Headers:Pin_Header_Straight_1x03_Pitch2.54mm, F.Cu at (33.0, 134.9)
- added J2: GPS, Pin_Headers:Pin_Header_Straight_1x03_Pitch2.54mm, F.Cu at (66.8, 135.2)
- added J2: GPS, Pin_Headers:Pin_Header_Straight_1x03_Pitch2.54mm, F.Cu at (140.7, 136.8)
- added J2: GPS, Pin_Headers:Pin_Header_Straight_1x03_Pitch2.54mm, F.Cu at (106.9, 136.4)
- added J2: GPS, Pin_Headers:Pin_Header_Straight_1x03_Pitch2.54mm, F.Cu at (106.9, 40.9)
- added J3: DHT, Pin_Headers:Pin_Header_Straight_1x04_Pitch2.54mm, F.Cu at (186.6, 35.2)
- added J3: DHT, Pin_Headers:Pin_Header_Straight_1x04_Pitch2.54mm, F.Cu at (141.3, 35.5)
- added J3: DHT, Pin_Headers:Pin_Header_Straight_1x04_Pitch2.54mm, F.Cu at (67.4, 34.0)
- added J3: DHT, Pin_Headers:Pin_Header_Straight_1x04_Pitch2.54mm, F.Cu at (220.3, 35.5)
- added J3: DHT, Pin_Headers:Pin_Header_Straight_1x04_Pitch2.54mm, F.Cu at (220.3, 131.0)
- added J3: DHT, Pin_Headers:Pin_Header_Straight_1x04_Pitch2.54mm, F.Cu at (186.6, 130.7)
- added J3: DHT, Pin_Headers:Pin_Header_Straight_1x04_Pitch2.54mm, F.Cu at (33.7, 129.2)
- added J3: DHT, Pin_Headers:Pin_Header_Straight_1x04_Pitch2.54mm, F.Cu at (67.4, 129.5)
- added J3: DHT, Pin_Headers:Pin_Header_Straight_1x04_Pitch2.54mm, F.Cu at (141.3, 131.0)
- added J3: DHT, Pin_Headers:Pin_Header_Straight_1x04_Pitch2.54mm, F.Cu at (107.6, 130.7)
- added J3: DHT, Pin_Headers:Pin_Header_Straight_1x04_Pitch2.54mm, F.Cu at (107.6, 35.2)
- added R1: R, Resistors_Universal:Resistor_SMD+THTuniversal_2512_RM10_HandSoldering_RevA_Date25Jun2010, F.Cu at (182.8, 30.1)
- added R1: R, Resistors_Universal:Resistor_SMD+THTuniversal_2512_RM10_HandSoldering_RevA_Date25Jun2010, F.Cu at (137.5, 30.5)
- added R1: R, Resistors_Universal:Resistor_SMD+THTuniversal_2512_RM10_HandSoldering_RevA_Date25Jun2010, F.Cu at (63.6, 28.9)
- added R1: R, Resistors_Universal:Resistor_SMD+THTuniversal_2512_RM10_HandSoldering_RevA_Date25Jun2010, F.Cu at (216.5, 30.5)
- added R1: R, Resistors_Universal:Resistor_SMD+THTuniversal_2512_RM10_HandSoldering_RevA_Date25Jun2010, F.Cu at (216.5, 126.0)
- added R1: R, Resistors_Universal:Resistor_SMD+THTuniversal_2512_RM10_HandSoldering_RevA_Date25Jun2010, F.Cu at (182.8, 125.6)
- added R1: R, Resistors_Universal:Resistor_SMD+THTuniversal_2512_RM10_HandSoldering_RevA_Date25Jun2010, F.Cu at (29.8, 124.1)
- added R1: R, Resistors_Universal:Resistor_SMD+THTuniversal_2512_RM10_HandSoldering_RevA_Date25Jun2010, F.Cu at (63.6, 124.4)
- added R1: R, Resistors_Universal:Resistor_SMD+THTuniversal_2512_RM10_HandSoldering_RevA_Date25Jun2010, F.Cu at (137.5, 126.0)
- added R1: R, Resistors_Universal:Resistor_SMD+THTuniversal_2512_RM10_HandSoldering_RevA_Date25Jun2010, F.Cu at (103.8, 125.6)
- added R1: R, Resistors_Universal:Resistor_SMD+THTuniversal_2512_RM10_HandSoldering_RevA_Date25Jun2010, F.Cu at (103.8, 30.1)
- added U1: UnloquerMCU_ver01, unloqueMCU_ver01_footprint:UnloquerMCU_ver01_footprint, F.Cu at (187.3, 40.5)
- added U1: UnloquerMCU_ver01, unloqueMCU_ver01_footprint:UnloquerMCU_ver01_footprint, F.Cu at (142.1, 40.9)
- added U1: UnloquerMCU_ver01, unloqueMCU_ver01_footprint:UnloquerMCU_ver01_footprint, F.Cu at (68.1, 39.4)
- added U1: UnloquerMCU_ver01, unloqueMCU_ver01_footprint:UnloquerMCU_ver01_footprint, F.Cu at (221.0, 40.9)
- added U1: UnloquerMCU_ver01, unloqueMCU_ver01_footprint:UnloquerMCU_ver01_footprint, F.Cu at (221.0, 136.4)
- added U1: UnloquerMCU_ver01, unloqueMCU_ver01_footprint:UnloquerMCU_ver01_footprint, F.Cu at (187.3, 136.0)
- added U1: UnloquerMCU_ver01, unloqueMCU_ver01_footprint:UnloquerMCU_ver01_footprint, F.Cu at (34.4, 134.5)
- added U1: UnloquerMCU_ver01, unloqueMCU_ver01_footprint:UnloquerMCU_ver01_footprint, F.Cu at (68.1, 134.9)
- added U1: UnloquerMCU_ver01, unloqueMCU_ver01_footprint:UnloquerMCU_ver01_footprint, F.Cu at (142.1, 136.4)
- added U1: UnloquerMCU_ver01, unloqueMCU_ver01_footprint:UnloquerMCU_ver01_footprint, F.Cu at (108.3, 136.0)
- added U1: UnloquerMCU_ver01, unloqueMCU_ver01_footprint:UnloquerMCU_ver01_footprint, F.Cu at (108.3, 40.5)
Connections:
- J1 pad 3: /gpio0 -> /gpio2
- J2 pad 1: +5V -> +3V3
- J2 pad 2: /gpio16 -> /gpio13
- J3 pad 1: +5V -> +3V3
- R1 pad 1: +5V -> +3V3
- U1 pad 12: Net-(U1-Pad12) -> +3V3
- U1 pad 13: Net-(U1-Pad13) -> /gpio13
- U1 pad 16: /gpio16 -> Net-(U1-Pad16)
- U1 pad 4: Net-(U1-Pad4) -> /gpio2
- U1 pad 5: /gpio0 -> Net-(U1-Pad5)
Routing:
- net +3V3: track 0.00 -> 357.4 mm
- net +5V: track 427.7 -> 120.3 mm
- net /gpio13: track 0.00 -> 179.1 mm
- net /gpio16: track 153.0 -> 0.00 mm
- net /gpio0: track 106.9 -> 0.00 mm
- net /gpio2: track 0.00 -> 76.0 mm
- net /gpio4: track 246.5 -> 227.5 mm
Other:
- board size 227.3 x 150.5 mm -> 217.1 x 134.2 mm
