File: proyectosKicad/calidadAirePlantTower/polvo_sensor_plant_tower.sch (KiCad schematic (older format))
At the start: 5 parts, among them J1 PLANTTOWER, J2 GPS, J3 DHT, U1 UnloquerMCU_ver01

Commit message: alimentacion y pines ok
Connections:
- net +5V: no longer J2.1 (P1), J3.1 (P1), R1.1
- net +3V3: now reaches U1.12 (+3.3V)
- net +3V3: now also J2.1 (P1), J3.1 (P1), R1.1
- net gpio13: now reaches U1.13 (GPIO13)
- net gpio13: now also J2.2 (P2)
- net gpio2: now reaches U1.4 (GPIO2)
- net gpio2: now also J1.3 (P3)
- net gpio0: no longer names the net of U1.5 (GPIO0)
- net gpio0: no longer J1.3 (P3)
- net gpio16: no longer names the net of U1.16 (GPIO16)
- net gpio16: no longer J2.2 (P2)
- no-connect marks 15 -> 14
Changed lines of the file:
@@
 $EndComp
 Text Label 5750 2550 2    60   ~ 0
-5vdc
+3.3vdc
 Text Label 6250 2850 0    60   ~ 0
 gpio4
@@
 ground
 Text Label 3750 2500 3    60   ~ 0
-5vdc
+3.3vdc
 Text Label 4550 3300 1    60   ~ 0
 gpio4
 Text Label 3850 2500 3    60   ~ 0
-gpio16
+gpio13
 Text Label 3950 2500 3    60   ~ 0
 ground
@@
 5vdc
 Text Label 3900 1800 3    60   ~ 0
-gpio0
+gpio2
 Text Label 3550 3300 1    60   ~ 0
 5vdc
@@
 Wire Wire Line
 	3700 4850 3700 4750
-NoConn ~ 3900 4750
-NoConn ~ 4050 4750
 NoConn ~ 4200 4750
 NoConn ~ 4500 4750
 NoConn ~ 3550 4750
 NoConn ~ 4900 4750
-NoConn ~ 4200 3550
 NoConn ~ 4050 3550
 NoConn ~ 3900 3550
-Text Label 4400 3300 1    60   ~ 0
-gpio0
+Text Label 4200 3350 1    60   ~ 0
+gpio2
+Text Label 4050 4900 3    60   ~ 0
+gpio13
+NoConn ~ 4700 3550
 Wire Wire Line
-	4400 3300 4400 3550
-Text Label 4650 4900 3    60   ~ 0
-gpio16
+	4200 3350 4200 3550
+NoConn ~ 4400 3550
+$Comp
+L PWR_FLAG #FLG05
+U 1 1 591A3D89
+P 7250 2500
+F 0 "#FLG05" H 7250 2575 50  0001 C CNN
+F 1 "PWR_FLAG" H 7250 2674 50  0000 C CNN
+F 2 "" H 7250 2500 50  0001 C CNN
+F 3 "" H 7250 2500 50  0001 C CNN
+	1    7250 2500
+	1    0    0    -1
+$EndComp
+$Comp
+L +3.3V #PWR06
+U 1 1 591A3DCF
+P 7250 2600
+F 0 "#PWR06" H 7250 2450 50  0001 C CNN
+F 1 "+3.3V" H 7265 2773 50  0000 C CNN
+F 2 "" H 7250 2600 50  0001 C CNN
+F 3 "" H 7250 2600 50  0001 C CNN
+	1    7250 2600
+	-1   0    0    1
+$EndComp
+Text Label 7050 2550 2    60   ~ 0
+3.3vdc
 Wire Wire Line
-	4650 4750 4650 4900
-NoConn ~ 4700 3550
+	7250 2500 7250 2600
+Wire Wire Line
+	7050 2550 7250 2550
+Connection ~ 7250 2550
+Text Label 3900 4900 3    60   ~ 0
+3.3vdc
+Wire Wire Line
+	3900 4900 3900 4750
+Wire Wire Line
+	4050 4750 4050 4900
+NoConn ~ 4650 4750
 $EndSCHEMATC
